File: Project 3 - BACEE.kicad_pcb (KiCad board)
At the start: 2 copper layers, 0 parts

Commit message: Set design rules.
Parts:
- added BT1: Battery 3V, Connector_PinHeader_2.54mm:PinHeader_1x02_P2.54mm_Vertical, F.Cu at (82.9, 86.1)
- added C1: 22pF, Capacitor_SMD:C_0805_2012Metric_Pad1.15x1.40mm_HandSolder, F.Cu at (132.4, 100.1)
- added C2: 22pF, Capacitor_SMD:C_0805_2012Metric_Pad1.15x1.40mm_HandSolder, F.Cu at (131.5, 107.3)
- added C3: 10uF, Capacitor_SMD:C_0805_2012Metric_Pad1.15x1.40mm_HandSolder, F.Cu at (126.8, 110.3)
- added D1: LED, LED_SMD:LED_0805_2012Metric_Pad1.15x1.40mm_HandSolder, F.Cu at (122.3, 102.3)
- added J1: Digital pins, Connector_PinSocket_2.54mm:PinSocket_1x09_P2.54mm_Vertical, F.Cu at (58.6, 84.9)
- added J2: Serial, Connector_PinSocket_2.54mm:PinSocket_1x04_P2.54mm_Vertical, F.Cu at (67.8, 84.9)
- added J3: ICSP, Connector_PinSocket_2.54mm:PinSocket_2x03_P2.54mm_Vertical, F.Cu at (74.9, 84.9)
- added J4: I2C, Connector_PinSocket_2.54mm:PinSocket_1x04_P2.54mm_Vertical, F.Cu at (63.2, 84.9)
- added R1: 330Ohm, Resistor_SMD:R_0805_2012Metric_Pad1.15x1.40mm_HandSolder, F.Cu at (132.4, 103.1)
- added R2: 10kOhm, Resistor_SMD:R_0805_2012Metric_Pad1.15x1.40mm_HandSolder, F.Cu at (126.8, 107.3)
- added U1: DS1337S, Package_SO:SO-8_5.3x6.2mm_P1.27mm, F.Cu at (119.2, 109.1)
- added U2: 24LC1025, Package_SO:SOIJ-8_5.3x5.3mm_P1.27mm, F.Cu at (120.1, 97.3)
- added U3: 24LC1025, Package_SO:SOIJ-8_5.3x5.3mm_P1.27mm, F.Cu at (108.7, 108.7)
- added U4: ATMEGA328P-AU, digikey-footprints:TQFP-32_7x7mm, F.Cu at (109.1, 99.5)
- added Y1: Crystal 32 MHz, Crystal:Crystal_SMD_MicroCrystal_CC7V-T1A-2Pin_3.2x1.5mm, F.Cu at (117.4, 102.5)
- added Y2: Crystal 16 MHz, Crystal:Crystal_SMD_5032-2Pin_5.0x3.2mm_HandSoldering, F.Cu at (130.5, 96.2)
Other:
- net class Power added: clearance 0.2, trace_width 0.3, via_dia 1, via_drill 0.6

Commit message: Placement complete.
Parts:
- moved R2 69.1 mm to (59.4, 91.9)
- moved Y2 68.4 mm to (62.1, 95.9)
- moved C1 62.8 mm to (69.6, 100.1)
- moved C2 62.8 mm to (69.6, 96.8)
- moved R1 48.7 mm to (84.1, 109.2)
- moved U2 44.4 mm to (76.7, 106.8)
- moved U4 43.9 mm to (65.8, 106.6)
- moved C3 43.1 mm to (84.0, 105.3)
- moved D1 34.1 mm to (88.9, 109.2)
- moved U1 34.1 mm to (87.0, 97.9)
- moved U3 33.7 mm to (76.7, 98.0)
- moved J1 32.1 mm to (66.3, 116.1), turned to 90 degrees
- moved BT1 29.9 mm to (54.6, 95.8)
- moved Y1 29.3 mm to (88.1, 105.0)
- moved J3 27.4 mm to (57.1, 105.8)
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
Commit message: Created outline and mounting holes.
Other:
- board outline added: 40.4 x 29.7 mm
Changed lines of the file:
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@@
   (general
     (thickness 1.6)
-    (drawings 0)
+    (drawings 12)
     (tracks 0)
     (zones 0)
@@
     )
   )
+  (gr_circle (center 90.424 116.84) (end 91.44 116.078) (layer Edge.Cuts) (width 0.05))
+  (gr_circle (center 90.424 90.678) (end 91.44 89.916) (layer Edge.Cuts) (width 0.05))
+  (gr_circle (center 53.594 116.84) (end 54.61 116.078) (layer Edge.Cuts) (width 0.05))
+  (gr_circle (center 53.594 90.678) (end 54.61 89.916) (layer Edge.Cuts) (width 0.05))
+  (gr_line (start 92.202 118.11) (end 92.202 89.408) (layer Edge.Cuts) (width 0.05))
+  (gr_line (start 52.324 118.618) (end 91.694 118.618) (layer Edge.Cuts) (width 0.05))
+  (gr_line (start 51.816 89.408) (end 51.816 118.11) (layer Edge.Cuts) (width 0.05))
+  (gr_line (start 91.694 88.9) (end 52.324 88.9) (layer Edge.Cuts) (width 0.05))
+  (gr_arc (start 91.694 89.408) (end 92.202 89.408) (angle -90) (layer Edge.Cuts) (width 0.05))
+  (gr_arc (start 91.694 118.11) (end 91.694 118.618) (angle -90) (layer Edge.Cuts) (width 0.05))
+  (gr_arc (start 52.324 118.11) (end 51.816 118.11) (angle -90) (layer Edge.Cuts) (width 0.05))
+  (gr_arc (start 52.324 89.408) (end 52.324 88.9) (angle -90) (layer Edge.Cuts) (width 0.05))
 )
